File: hardware/TIYCS_ledPanel/TIYCS_ledPanel.kicad_pcb (KiCad board)
At the start: 2 copper layers, 100 x 100 mm, 108 parts

Commit message: Routed
Parts:
- removed the R_0_0_RGB at (-35.0, -30.0)
- removed the R_0_1_RGB at (-35.0, -32.0)
- removed the R_0_2_RGB at (-35.0, -28.0)
- removed the R_3_0_RGB at (30.0, -35.0)
- removed the R_3_1_RGB at (32.0, -35.0)
- removed the R_3_2_RGB at (28.0, -35.0)
- removed the R_6_0_RGB at (35.0, 30.0)
- removed the R_6_1_RGB at (35.0, 32.0)
- removed the R_6_2_RGB at (35.0, 28.0)
- removed the R_9_0_RGB at (-30.0, 35.0)
- removed the R_9_1_RGB at (-32.0, 35.0)
- removed the R_9_2_RGB at (-28.0, 35.0)
- added R_0_0_RGB2: R_0603_1608Metric, R_0603_1608Metric, F.Cu at (-35.0, -30.0)
- added R_0_1_RGB2: R_0603_1608Metric, R_0603_1608Metric, F.Cu at (-35.0, -32.0)
- added R_0_2_RGB2: R_0603_1608Metric, R_0603_1608Metric, F.Cu at (-35.0, -28.0)
- added R_3_0_RGB2: R_0603_1608Metric, R_0603_1608Metric, F.Cu at (30.0, -35.0)
- added R_3_1_RGB2: R_0603_1608Metric, R_0603_1608Metric, F.Cu at (32.0, -35.0)
- added R_3_2_RGB2: R_0603_1608Metric, R_0603_1608Metric, F.Cu at (28.0, -35.0)
- added R_6_0_RGB2: R_0603_1608Metric, R_0603_1608Metric, F.Cu at (35.0, 30.0)
- added R_6_1_RGB2: R_0603_1608Metric, R_0603_1608Metric, F.Cu at (35.0, 32.0)
- added R_6_2_RGB2: R_0603_1608Metric, R_0603_1608Metric, F.Cu at (35.0, 28.0)
- added R_9_0_RGB2: R_0603_1608Metric, R_0603_1608Metric, F.Cu at (-30.0, 35.0)
- added R_9_1_RGB2: R_0603_1608Metric, R_0603_1608Metric, F.Cu at (-32.0, 35.0)
- added R_9_2_RGB2: R_0603_1608Metric, R_0603_1608Metric, F.Cu at (-28.0, 35.0)
Connections:
- net D10toD11_W renamed D10toD11_W_1
- net D12toD13_Blue renamed D12toD13_Blue_1
- net D12toD13_Green renamed D12toD13_Green_1
- net D12toD13_Red renamed D12toD13_Red_1
- net D13toD14_Blue renamed D13toD14_Blue_1
- net D13toD14_Green renamed D13toD14_Green_1
- net D13toD14_Red renamed D13toD14_Red_1
- net D15toD16_Blue renamed D15toD16_Blue_1
- net D15toD16_Green renamed D15toD16_Green_1
- net D15toD16_Red renamed D15toD16_Red_1
- net D16toD17_Blue renamed D16toD17_Blue_1
- net D16toD17_Green renamed D16toD17_Green_1
- net D16toD17_Red renamed D16toD17_Red_1
- net D18toD19_Blue renamed D18toD19_Blue_1
- net D18toD19_Green renamed D18toD19_Green_1
- net D18toD19_Red renamed D18toD19_Red_1
- net D19toD20_Blue renamed D19toD20_Blue_1
- net D19toD20_Green renamed D19toD20_Green_1
- net D19toD20_Red renamed D19toD20_Red_1
- net D21toD22_Blue renamed D21toD22_Blue_1
- net D21toD22_Green renamed D21toD22_Green_1
- net D21toD22_Red renamed D21toD22_Red_1
- net D22toD23_Blue renamed D22toD23_Blue_1
- net D22toD23_Green renamed D22toD23_Green_1
- net D22toD23_Red renamed D22toD23_Red_1
- net D4toD5_W renamed D4toD5_W_1
- net D6toD7_W renamed D6toD7_W_1
- net D8toD9_W renamed D8toD9_W_1
- net RtoD10_W renamed RtoD10_W_1
- net RtoD12_Blue renamed RtoD12_Blue_1
- net RtoD12_Green renamed RtoD12_Green_1
- net RtoD12_Red renamed RtoD12_Red_1
- net RtoD15_Blue renamed RtoD15_Blue_1
- net RtoD15_Green renamed RtoD15_Green_1
- net RtoD15_Red renamed RtoD15_Red_1
- net RtoD18_Blue renamed RtoD18_Blue_1
- net RtoD18_Green renamed RtoD18_Green_1
- net RtoD18_Red renamed RtoD18_Red_1
- net RtoD21_Blue renamed RtoD21_Blue_1
- net RtoD21_Green renamed RtoD21_Green_1
- net RtoD21_Red renamed RtoD21_Red_1
- net RtoD4_W renamed RtoD4_W_1
- net RtoD6_W renamed RtoD6_W_1
- net RtoD8_W renamed RtoD8_W_1
- LED_RGB2_0 pad 1: RtoD0_Green -> RtoD0_Green_2
- LED_RGB2_0 pad 2: RtoD0_Red -> RtoD0_Red_2
- LED_RGB2_0 pad 3: RtoD0_Blue -> RtoD0_Blue_2
- LED_RGB2_0 pad 4: D0toD1_Blue -> D0toD1_Blue_2
- LED_RGB2_0 pad 5: D0toD1_Red -> D0toD1_Red_2
- LED_RGB2_0 pad 6: D0toD1_Green -> D0toD1_Green_2
- LED_RGB2_1 pad 1: D0toD1_Green -> D0toD1_Green_2
- LED_RGB2_1 pad 2: D0toD1_Red -> D0toD1_Red_2
- LED_RGB2_1 pad 3: D0toD1_Blue -> D0toD1_Blue_2
- LED_RGB2_1 pad 4: D1toD2_Blue -> D1toD2_Blue_2
- LED_RGB2_1 pad 5: D1toD2_Red -> D1toD2_Red_2
- LED_RGB2_1 pad 6: D1toD2_Green -> D1toD2_Green_2
- LED_RGB2_10 pad 1: D9toD10_Green -> D9toD10_Green_2
- LED_RGB2_10 pad 2: D9toD10_Red -> D9toD10_Red_2
- LED_RGB2_10 pad 3: D9toD10_Blue -> D9toD10_Blue_2
- LED_RGB2_10 pad 4: D10toD11_Blue -> D10toD11_Blue_2
- LED_RGB2_10 pad 5: D10toD11_Red -> D10toD11_Red_2
- LED_RGB2_10 pad 6: D10toD11_Green -> D10toD11_Green_2
- LED_RGB2_11 pad 1: D10toD11_Green -> D10toD11_Green_2
- LED_RGB2_11 pad 2: D10toD11_Red -> D10toD11_Red_2
- LED_RGB2_11 pad 3: D10toD11_Blue -> D10toD11_Blue_2
- LED_RGB2_2 pad 1: D1toD2_Green -> D1toD2_Green_2
- LED_RGB2_2 pad 2: D1toD2_Red -> D1toD2_Red_2
- LED_RGB2_2 pad 3: D1toD2_Blue -> D1toD2_Blue_2
- LED_RGB2_3 pad 1: RtoD3_Green -> RtoD3_Green_2
- LED_RGB2_3 pad 2: RtoD3_Red -> RtoD3_Red_2
- LED_RGB2_3 pad 3: RtoD3_Blue -> RtoD3_Blue_2
- LED_RGB2_3 pad 4: D3toD4_Blue -> D3toD4_Blue_2
- LED_RGB2_3 pad 5: D3toD4_Red -> D3toD4_Red_2
- LED_RGB2_3 pad 6: D3toD4_Green -> D3toD4_Green_2
- LED_RGB2_4 pad 1: D3toD4_Green -> D3toD4_Green_2
- LED_RGB2_4 pad 2: D3toD4_Red -> D3toD4_Red_2
- LED_RGB2_4 pad 3: D3toD4_Blue -> D3toD4_Blue_2
- LED_RGB2_4 pad 4: D4toD5_Blue -> D4toD5_Blue_2
- LED_RGB2_4 pad 5: D4toD5_Red -> D4toD5_Red_2
- LED_RGB2_4 pad 6: D4toD5_Green -> D4toD5_Green_2
- LED_RGB2_5 pad 1: D4toD5_Green -> D4toD5_Green_2
- LED_RGB2_5 pad 2: D4toD5_Red -> D4toD5_Red_2
- LED_RGB2_5 pad 3: D4toD5_Blue -> D4toD5_Blue_2
- LED_RGB2_6 pad 1: RtoD6_Green -> RtoD6_Green_2
- LED_RGB2_6 pad 2: RtoD6_Red -> RtoD6_Red_2
- LED_RGB2_6 pad 3: RtoD6_Blue -> RtoD6_Blue_2
- LED_RGB2_6 pad 4: D6toD7_Blue -> D6toD7_Blue_2
- LED_RGB2_6 pad 5: D6toD7_Red -> D6toD7_Red_2
- LED_RGB2_6 pad 6: D6toD7_Green -> D6toD7_Green_2
- LED_RGB2_7 pad 1: D6toD7_Green -> D6toD7_Green_2
- LED_RGB2_7 pad 2: D6toD7_Red -> D6toD7_Red_2
- LED_RGB2_7 pad 3: D6toD7_Blue -> D6toD7_Blue_2
- LED_RGB2_7 pad 4: D7toD8_Blue -> D7toD8_Blue_2
- LED_RGB2_7 pad 5: D7toD8_Red -> D7toD8_Red_2
- LED_RGB2_7 pad 6: D7toD8_Green -> D7toD8_Green_2
- LED_RGB2_8 pad 1: D7toD8_Green -> D7toD8_Green_2
- LED_RGB2_8 pad 2: D7toD8_Red -> D7toD8_Red_2
- LED_RGB2_8 pad 3: D7toD8_Blue -> D7toD8_Blue_2
- LED_RGB2_9 pad 1: RtoD9_Green -> RtoD9_Green_2
- LED_RGB2_9 pad 2: RtoD9_Red -> RtoD9_Red_2
- LED_RGB2_9 pad 3: RtoD9_Blue -> RtoD9_Blue_2
- LED_RGB2_9 pad 4: D9toD10_Blue -> D9toD10_Blue_2
- LED_RGB2_9 pad 5: D9toD10_Red -> D9toD10_Red_2
- LED_RGB2_9 pad 6: D9toD10_Green -> D9toD10_Green_2
- LED_RGB_0 pad 1: RtoD0_Green -> RtoD0_Green_1
- LED_RGB_0 pad 2: RtoD0_Red -> RtoD0_Red_1
- LED_RGB_0 pad 3: RtoD0_Blue -> RtoD0_Blue_1
- LED_RGB_0 pad 4: D0toD1_Blue -> D0toD1_Blue_1
- LED_RGB_0 pad 5: D0toD1_Red -> D0toD1_Red_1
- LED_RGB_0 pad 6: D0toD1_Green -> D0toD1_Green_1
- LED_RGB_1 pad 1: D0toD1_Green -> D0toD1_Green_1
- LED_RGB_1 pad 2: D0toD1_Red -> D0toD1_Red_1
- LED_RGB_1 pad 3: D0toD1_Blue -> D0toD1_Blue_1
- LED_RGB_1 pad 4: D1toD2_Blue -> D1toD2_Blue_1
- LED_RGB_1 pad 5: D1toD2_Red -> D1toD2_Red_1
- LED_RGB_1 pad 6: D1toD2_Green -> D1toD2_Green_1
- LED_RGB_10 pad 1: D9toD10_Green -> D9toD10_Green_1
- LED_RGB_10 pad 2: D9toD10_Red -> D9toD10_Red_1
- LED_RGB_10 pad 3: D9toD10_Blue -> D9toD10_Blue_1
- LED_RGB_10 pad 4: D10toD11_Blue -> D10toD11_Blue_1
- LED_RGB_10 pad 5: D10toD11_Red -> D10toD11_Red_1
- LED_RGB_10 pad 6: D10toD11_Green -> D10toD11_Green_1
- LED_RGB_11 pad 1: D10toD11_Green -> D10toD11_Green_1
- LED_RGB_11 pad 2: D10toD11_Red -> D10toD11_Red_1
- LED_RGB_11 pad 3: D10toD11_Blue -> D10toD11_Blue_1
- LED_RGB_2 pad 1: D1toD2_Green -> D1toD2_Green_1
- LED_RGB_2 pad 2: D1toD2_Red -> D1toD2_Red_1
- LED_RGB_2 pad 3: D1toD2_Blue -> D1toD2_Blue_1
- LED_RGB_3 pad 1: RtoD3_Green -> RtoD3_Green_1
- LED_RGB_3 pad 2: RtoD3_Red -> RtoD3_Red_1
- LED_RGB_3 pad 3: RtoD3_Blue -> RtoD3_Blue_1
- LED_RGB_3 pad 4: D3toD4_Blue -> D3toD4_Blue_1
- LED_RGB_3 pad 5: D3toD4_Red -> D3toD4_Red_1
- LED_RGB_3 pad 6: D3toD4_Green -> D3toD4_Green_1
- LED_RGB_4 pad 1: D3toD4_Green -> D3toD4_Green_1
- LED_RGB_4 pad 2: D3toD4_Red -> D3toD4_Red_1
- LED_RGB_4 pad 3: D3toD4_Blue -> D3toD4_Blue_1
- LED_RGB_4 pad 4: D4toD5_Blue -> D4toD5_Blue_1
- LED_RGB_4 pad 5: D4toD5_Red -> D4toD5_Red_1
- LED_RGB_4 pad 6: D4toD5_Green -> D4toD5_Green_1
- LED_RGB_5 pad 1: D4toD5_Green -> D4toD5_Green_1
- LED_RGB_5 pad 2: D4toD5_Red -> D4toD5_Red_1
- LED_RGB_5 pad 3: D4toD5_Blue -> D4toD5_Blue_1
- LED_RGB_6 pad 1: RtoD6_Green -> RtoD6_Green_1
- LED_RGB_6 pad 2: RtoD6_Red -> RtoD6_Red_1
- LED_RGB_6 pad 3: RtoD6_Blue -> RtoD6_Blue_1
- LED_RGB_6 pad 4: D6toD7_Blue -> D6toD7_Blue_1
- LED_RGB_6 pad 5: D6toD7_Red -> D6toD7_Red_1
- LED_RGB_6 pad 6: D6toD7_Green -> D6toD7_Green_1
- LED_RGB_7 pad 1: D6toD7_Green -> D6toD7_Green_1
- LED_RGB_7 pad 2: D6toD7_Red -> D6toD7_Red_1
- LED_RGB_7 pad 3: D6toD7_Blue -> D6toD7_Blue_1
- LED_RGB_7 pad 4: D7toD8_Blue -> D7toD8_Blue_1
- LED_RGB_7 pad 5: D7toD8_Red -> D7toD8_Red_1
- LED_RGB_7 pad 6: D7toD8_Green -> D7toD8_Green_1
- LED_RGB_8 pad 1: D7toD8_Green -> D7toD8_Green_1
- LED_RGB_8 pad 2: D7toD8_Red -> D7toD8_Red_1
- LED_RGB_8 pad 3: D7toD8_Blue -> D7toD8_Blue_1
- LED_RGB_9 pad 1: RtoD9_Green -> RtoD9_Green_1
- LED_RGB_9 pad 2: RtoD9_Red -> RtoD9_Red_1
- LED_RGB_9 pad 3: RtoD9_Blue -> RtoD9_Blue_1
- LED_RGB_9 pad 4: D9toD10_Blue -> D9toD10_Blue_1
- LED_RGB_9 pad 5: D9toD10_Red -> D9toD10_Red_1
- LED_RGB_9 pad 6: D9toD10_Green -> D9toD10_Green_1
- LED_W2_0 pad 1: RtoD0_W -> RtoD0_W_2
- LED_W2_0 pad 2: RtoD0_W -> RtoD0_W_2
- LED_W2_0 pad 3: RtoD0_W -> RtoD0_W_2
- LED_W2_0 pad 4: D0toD1_W -> D0toD1_W_2
- LED_W2_0 pad 5: D0toD1_W -> D0toD1_W_2
- LED_W2_0 pad 6: D0toD1_W -> D0toD1_W_2
- LED_W2_1 pad 1: D0toD1_W -> D0toD1_W_2
- LED_W2_1 pad 2: D0toD1_W -> D0toD1_W_2
- LED_W2_1 pad 3: D0toD1_W -> D0toD1_W_2
- LED_W2_2 pad 1: RtoD2_W -> RtoD2_W_2
- LED_W2_2 pad 2: RtoD2_W -> RtoD2_W_2
- LED_W2_2 pad 3: RtoD2_W -> RtoD2_W_2
- LED_W2_2 pad 4: D2toD3_W -> D2toD3_W_2
- LED_W2_2 pad 5: D2toD3_W -> D2toD3_W_2
- LED_W2_2 pad 6: D2toD3_W -> D2toD3_W_2
- LED_W2_3 pad 1: D2toD3_W -> D2toD3_W_2
- LED_W2_3 pad 2: D2toD3_W -> D2toD3_W_2
- LED_W2_3 pad 3: D2toD3_W -> D2toD3_W_2
- LED_W_0 pad 1: RtoD0_W -> RtoD0_W_1
- LED_W_0 pad 2: RtoD0_W -> RtoD0_W_1
- LED_W_0 pad 3: RtoD0_W -> RtoD0_W_1
- LED_W_0 pad 4: D0toD1_W -> D0toD1_W_1
- LED_W_0 pad 5: D0toD1_W -> D0toD1_W_1
- LED_W_0 pad 6: D0toD1_W -> D0toD1_W_1
- LED_W_1 pad 1: D0toD1_W -> D0toD1_W_1
- LED_W_1 pad 2: D0toD1_W -> D0toD1_W_1
- LED_W_1 pad 3: D0toD1_W -> D0toD1_W_1
- LED_W_2 pad 1: RtoD2_W -> RtoD2_W_1
- LED_W_2 pad 2: RtoD2_W -> RtoD2_W_1
- LED_W_2 pad 3: RtoD2_W -> RtoD2_W_1
- LED_W_2 pad 4: D2toD3_W -> D2toD3_W_1
- LED_W_2 pad 5: D2toD3_W -> D2toD3_W_1
- LED_W_2 pad 6: D2toD3_W -> D2toD3_W_1
- LED_W_3 pad 1: D2toD3_W -> D2toD3_W_1
- LED_W_3 pad 2: D2toD3_W -> D2toD3_W_1
- LED_W_3 pad 3: D2toD3_W -> D2toD3_W_1
- R_0_0_RGB pad 2: RtoD0_Red -> RtoD0_Red_1
- R_0_0_W pad 2: RtoD0_W -> RtoD0_W_1
- R_0_0_W2 pad 2: RtoD0_W -> RtoD0_W_2
- R_0_1_RGB pad 2: RtoD0_Green -> RtoD0_Green_1
- R_0_2_RGB pad 2: RtoD0_Blue -> RtoD0_Blue_1
- R_2_0_W pad 2: RtoD2_W -> RtoD2_W_1
- R_2_0_W2 pad 2: RtoD2_W -> RtoD2_W_2
- R_3_0_RGB pad 2: RtoD3_Red -> RtoD3_Red_1
- R_3_1_RGB pad 2: RtoD3_Green -> RtoD3_Green_1
- R_3_2_RGB pad 2: RtoD3_Blue -> RtoD3_Blue_1
- R_6_0_RGB pad 2: RtoD6_Red -> RtoD6_Red_1
- R_6_1_RGB pad 2: RtoD6_Green -> RtoD6_Green_1
- R_6_2_RGB pad 2: RtoD6_Blue -> RtoD6_Blue_1
- R_9_0_RGB pad 2: RtoD9_Red -> RtoD9_Red_1
- R_9_1_RGB pad 2: RtoD9_Green -> RtoD9_Green_1
- R_9_2_RGB pad 2: RtoD9_Blue -> RtoD9_Blue_1
Routing:
- net 12V: track 0.00 -> 627.5 mm, vias 0 -> 3
- net B: track 0.00 -> 469.9 mm, vias 0 -> 11
- net G: track 0.00 -> 467.2 mm, vias 0 -> 9
- net W: track 0.00 -> 440.6 mm, vias 0 -> 3
- net R: track 0.00 -> 422.9 mm, vias 0 -> 10
- net D2toD3_W_2: track 0.00 -> 23.9 mm
- net D0toD1_W_2: track 0.00 -> 23.8 mm
- net D2toD3_W_1: track 0.00 -> 22.8 mm
- net D8toD9_W_1: track 0.00 -> 21.9 mm
- net D10toD11_W_1: track 0.00 -> 21.8 mm
- net D0toD1_W_1: track 0.00 -> 21.8 mm
- net D6toD7_W_1: track 0.00 -> 21.8 mm
- net D4toD5_W_1: track 0.00 -> 19.2 mm
- net D4toD5_Blue_2: track 0.00 -> 15.4 mm
- net D9toD10_Red_2: track 0.00 -> 15.2 mm
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
Commit message: Panelization edge-cuts
Parts:
- removed H_0, H_1, H_2, H_3: MountingHole_3mm_Pad, MountingHole_3mm_Pad
- removed LED_RGB2_0, LED_RGB2_1, LED_RGB2_10, LED_RGB2_11, LED_RGB2_2, LED_RGB2_3, LED_RGB2_4, LED_RGB2_5, LED_RGB2_6, LED_RGB2_7, LED_RGB2_8, LED_RGB2_9, LED_RGB_0, LED_RGB_1, LED_RGB_10, LED_RGB_11, LED_RGB_12, LED_RGB_13, LED_RGB_14, LED_RGB_15, LED_RGB_16, LED_RGB_17, LED_RGB_18, LED_RGB_19, LED_RGB_2, LED_RGB_20, LED_RGB_21, LED_RGB_22, LED_RGB_23, LED_RGB_3, LED_RGB_4, LED_RGB_5, LED_RGB_6, LED_RGB_7, LED_RGB_8, LED_RGB_9, LED_W2_0, LED_W2_1, LED_W2_2, LED_W2_3, LED_W_0, LED_W_1, LED_W_10, LED_W_11, LED_W_2, LED_W_3, LED_W_4, LED_W_5, LED_W_6, LED_W_7, LED_W_8, LED_W_9: LED_RGB_5050-6, LED_RGB_5050-6
- removed R_0_0_RGB, R_0_0_RGB2, R_0_0_W, R_0_0_W2, R_0_1_RGB, R_0_1_RGB2, R_0_2_RGB, R_0_2_RGB2, R_10_0_W, R_12_0_RGB, R_12_1_RGB, R_12_2_RGB, R_15_0_RGB, R_15_1_RGB, R_15_2_RGB, R_18_0_RGB, R_18_1_RGB, R_18_2_RGB, R_21_0_RGB, R_21_1_RGB, R_21_2_RGB, R_2_0_W, R_2_0_W2, R_3_0_RGB, R_3_0_RGB2, R_3_1_RGB, R_3_1_RGB2, R_3_2_RGB, R_3_2_RGB2, R_4_0_W, R_6_0_RGB, R_6_0_RGB2, R_6_0_W, R_6_1_RGB, R_6_1_RGB2, R_6_2_RGB, R_6_2_RGB2, R_8_0_W, R_9_0_RGB, R_9_0_RGB2, R_9_1_RGB, R_9_1_RGB2, R_9_2_RGB, R_9_2_RGB2: R_0603_1608Metric, R_0603_1608Metric
- removed mainConn_0_0, mainConn_0_1, mainConn_1_0, mainConn_1_1, mainConn_2_0, mainConn_2_1, mainConn_3_0, mainConn_3_1: PinHeader_1x11_P2.54mm_Vertical, PinHeader_1x11_P2.54mm_Vertical
Routing:
- net 12V: track 627.5 -> 0.00 mm, vias 3 -> 0
- net B: track 469.9 -> 0.00 mm, vias 11 -> 0
- net G: track 467.2 -> 0.00 mm, vias 9 -> 0
- net W: track 440.6 -> 0.00 mm, vias 3 -> 0
- net R: track 422.9 -> 0.00 mm, vias 10 -> 0
- net D2toD3_W_2: track 23.9 -> 0.00 mm
- net D0toD1_W_2: track 23.8 -> 0.00 mm
- net D2toD3_W_1: track 22.8 -> 0.00 mm
- net D8toD9_W_1: track 21.9 -> 0.00 mm
- net D10toD11_W_1: track 21.8 -> 0.00 mm
- net D0toD1_W_1: track 21.8 -> 0.00 mm
- net D6toD7_W_1: track 21.8 -> 0.00 mm
- net D4toD5_W_1: track 19.2 -> 0.00 mm
- net D4toD5_Blue_2: track 15.4 -> 0.00 mm
- net D9toD10_Red_2: track 15.2 -> 0.00 mm
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Other:
- board outline removed

Commit message: Routed battery PCB
Parts:
- added H_0: MountingHole_3mm_Pad, MountingHole_3mm_Pad, F.Cu at (-46.0, -46.0)
- added H_1: MountingHole_3mm_Pad, MountingHole_3mm_Pad, F.Cu at (46.0, -46.0)
- added H_10: MountingHole_3mm_Pad, MountingHole_3mm_Pad, F.Cu at (46.0, 149.0)
- added H_11: MountingHole_3mm_Pad, MountingHole_3mm_Pad, F.Cu at (-46.0, 149.0)
- added H_12: MountingHole_3mm_Pad, MountingHole_3mm_Pad, F.Cu at (57.0, 57.0)
- added H_13: MountingHole_3mm_Pad, MountingHole_3mm_Pad, F.Cu at (149.0, 57.0)
- added H_14: MountingHole_3mm_Pad, MountingHole_3mm_Pad, F.Cu at (149.0, 149.0)
- added H_15: MountingHole_3mm_Pad, MountingHole_3mm_Pad, F.Cu at (57.0, 149.0)
- added H_2: MountingHole_3mm_Pad, MountingHole_3mm_Pad, F.Cu at (46.0, 46.0)
- added H_3: MountingHole_3mm_Pad, MountingHole_3mm_Pad, F.Cu at (-46.0, 46.0)
- added H_4: MountingHole_3mm_Pad, MountingHole_3mm_Pad, F.Cu at (57.0, -46.0)
- added H_5: MountingHole_3mm_Pad, MountingHole_3mm_Pad, F.Cu at (149.0, -46.0)
- added H_6: MountingHole_3mm_Pad, MountingHole_3mm_Pad, F.Cu at (149.0, 46.0)
- added H_7: MountingHole_3mm_Pad, MountingHole_3mm_Pad, F.Cu at (57.0, 46.0)
- added H_8: MountingHole_3mm_Pad, MountingHole_3mm_Pad, F.Cu at (-46.0, 57.0)
- added H_9: MountingHole_3mm_Pad, MountingHole_3mm_Pad, F.Cu at (46.0, 57.0)
- added LED_RGB2_0: LED_RGB_5050-6, LED_RGB_5050-6, F.Cu at (-29.0, -30.0)
- added LED_RGB2_1: LED_RGB_5050-6, LED_RGB_5050-6, F.Cu at (-9.00, -30.0)
- added LED_RGB2_10: LED_RGB_5050-6, LED_RGB_5050-6, F.Cu at (-30.0, 9.00)
- added LED_RGB2_11: LED_RGB_5050-6, LED_RGB_5050-6, F.Cu at (-30.0, -11.0)
- added LED_RGB2_12: LED_RGB_5050-6, LED_RGB_5050-6, F.Cu at (74.0, -30.0)
- added LED_RGB2_13: LED_RGB_5050-6, LED_RGB_5050-6, F.Cu at (94.0, -30.0)
- added LED_RGB2_14: LED_RGB_5050-6, LED_RGB_5050-6, F.Cu at (114.0, -30.0)
- added LED_RGB2_15: LED_RGB_5050-6, LED_RGB_5050-6, F.Cu at (133.0, -29.0)
- added LED_RGB2_16: LED_RGB_5050-6, LED_RGB_5050-6, F.Cu at (133.0, -9.00)
- added LED_RGB2_17: LED_RGB_5050-6, LED_RGB_5050-6, F.Cu at (133.0, 11.0)
- added LED_RGB2_18: LED_RGB_5050-6, LED_RGB_5050-6, F.Cu at (132.0, 30.0)
- added LED_RGB2_19: LED_RGB_5050-6, LED_RGB_5050-6, F.Cu at (112.0, 30.0)
- added LED_RGB2_2: LED_RGB_5050-6, LED_RGB_5050-6, F.Cu at (11.0, -30.0)
- added LED_RGB2_20: LED_RGB_5050-6, LED_RGB_5050-6, F.Cu at (92.0, 30.0)
- added LED_RGB2_21: LED_RGB_5050-6, LED_RGB_5050-6, F.Cu at (73.0, 29.0)
- added LED_RGB2_22: LED_RGB_5050-6, LED_RGB_5050-6, F.Cu at (73.0, 9.00)
- added LED_RGB2_23: LED_RGB_5050-6, LED_RGB_5050-6, F.Cu at (73.0, -11.0)
- added LED_RGB2_24: LED_RGB_5050-6, LED_RGB_5050-6, F.Cu at (-29.0, 73.0)
- added LED_RGB2_25: LED_RGB_5050-6, LED_RGB_5050-6, F.Cu at (-9.00, 73.0)
- added LED_RGB2_26: LED_RGB_5050-6, LED_RGB_5050-6, F.Cu at (11.0, 73.0)
- added LED_RGB2_27: LED_RGB_5050-6, LED_RGB_5050-6, F.Cu at (30.0, 74.0)
- added LED_RGB2_28: LED_RGB_5050-6, LED_RGB_5050-6, F.Cu at (30.0, 94.0)
- added LED_RGB2_29: LED_RGB_5050-6, LED_RGB_5050-6, F.Cu at (30.0, 114.0)
- added LED_RGB2_3: LED_RGB_5050-6, LED_RGB_5050-6, F.Cu at (30.0, -29.0)
- added LED_RGB2_30: LED_RGB_5050-6, LED_RGB_5050-6, F.Cu at (29.0, 133.0)
- added LED_RGB2_31: LED_RGB_5050-6, LED_RGB_5050-6, F.Cu at (9.00, 133.0)
- added LED_RGB2_32: LED_RGB_5050-6, LED_RGB_5050-6, F.Cu at (-11.0, 133.0)
- added LED_RGB2_33: LED_RGB_5050-6, LED_RGB_5050-6, F.Cu at (-30.0, 132.0)
- added LED_RGB2_34: LED_RGB_5050-6, LED_RGB_5050-6, F.Cu at (-30.0, 112.0)
- added LED_RGB2_35: LED_RGB_5050-6, LED_RGB_5050-6, F.Cu at (-30.0, 92.0)
- added LED_RGB2_36: LED_RGB_5050-6, LED_RGB_5050-6, F.Cu at (74.0, 73.0)
- added LED_RGB2_37: LED_RGB_5050-6, LED_RGB_5050-6, F.Cu at (94.0, 73.0)
- added LED_RGB2_38: LED_RGB_5050-6, LED_RGB_5050-6, F.Cu at (114.0, 73.0)
- added LED_RGB2_39: LED_RGB_5050-6, LED_RGB_5050-6, F.Cu at (133.0, 74.0)
- added LED_RGB2_4: LED_RGB_5050-6, LED_RGB_5050-6, F.Cu at (30.0, -9.00)
- added LED_RGB2_40: LED_RGB_5050-6, LED_RGB_5050-6, F.Cu at (133.0, 94.0)
- added LED_RGB2_41: LED_RGB_5050-6, LED_RGB_5050-6, F.Cu at (133.0, 114.0)
- added LED_RGB2_42: LED_RGB_5050-6, LED_RGB_5050-6, F.Cu at (132.0, 133.0)
- added LED_RGB2_43: LED_RGB_5050-6, LED_RGB_5050-6, F.Cu at (112.0, 133.0)
- added LED_RGB2_44: LED_RGB_5050-6, LED_RGB_5050-6, F.Cu at (92.0, 133.0)
- added LED_RGB2_45: LED_RGB_5050-6, LED_RGB_5050-6, F.Cu at (73.0, 132.0)
- added LED_RGB2_46: LED_RGB_5050-6, LED_RGB_5050-6, F.Cu at (73.0, 112.0)
- added LED_RGB2_47: LED_RGB_5050-6, LED_RGB_5050-6, F.Cu at (73.0, 92.0)
- added LED_RGB2_5: LED_RGB_5050-6, LED_RGB_5050-6, F.Cu at (30.0, 11.0)
- added LED_RGB2_6: LED_RGB_5050-6, LED_RGB_5050-6, F.Cu at (29.0, 30.0)
- added LED_RGB2_7: LED_RGB_5050-6, LED_RGB_5050-6, F.Cu at (9.00, 30.0)
- added LED_RGB2_8: LED_RGB_5050-6, LED_RGB_5050-6, F.Cu at (-11.0, 30.0)
- added LED_RGB2_9: LED_RGB_5050-6, LED_RGB_5050-6, F.Cu at (-30.0, 29.0)
- added LED_RGB_0: LED_RGB_5050-6, LED_RGB_5050-6, F.Cu at (-39.0, -40.0)
- added LED_RGB_1: LED_RGB_5050-6, LED_RGB_5050-6, F.Cu at (-25.7, -40.0)
- added LED_RGB_10: LED_RGB_5050-6, LED_RGB_5050-6, F.Cu at (40.0, 14.3)
- added LED_RGB_11: LED_RGB_5050-6, LED_RGB_5050-6, F.Cu at (40.0, 27.7)
- added LED_RGB_12: LED_RGB_5050-6, LED_RGB_5050-6, F.Cu at (39.0, 40.0)
- added LED_RGB_13: LED_RGB_5050-6, LED_RGB_5050-6, F.Cu at (25.7, 40.0)
- added LED_RGB_14: LED_RGB_5050-6, LED_RGB_5050-6, F.Cu at (12.3, 40.0)
- added LED_RGB_15: LED_RGB_5050-6, LED_RGB_5050-6, F.Cu at (-1.00, 40.0)
- added LED_RGB_16: LED_RGB_5050-6, LED_RGB_5050-6, F.Cu at (-14.3, 40.0)
- added LED_RGB_17: LED_RGB_5050-6, LED_RGB_5050-6, F.Cu at (-27.7, 40.0)
- added LED_RGB_18: LED_RGB_5050-6, LED_RGB_5050-6, F.Cu at (-40.0, 39.0)
- added LED_RGB_19: LED_RGB_5050-6, LED_RGB_5050-6, F.Cu at (-40.0, 25.7)
- added LED_RGB_2: LED_RGB_5050-6, LED_RGB_5050-6, F.Cu at (-12.3, -40.0)
- added LED_RGB_20: LED_RGB_5050-6, LED_RGB_5050-6, F.Cu at (-40.0, 12.3)
- added LED_RGB_21: LED_RGB_5050-6, LED_RGB_5050-6, F.Cu at (-40.0, -1.00)
- added LED_RGB_22: LED_RGB_5050-6, LED_RGB_5050-6, F.Cu at (-40.0, -14.3)
- added LED_RGB_23: LED_RGB_5050-6, LED_RGB_5050-6, F.Cu at (-40.0, -27.7)
- added LED_RGB_24: LED_RGB_5050-6, LED_RGB_5050-6, F.Cu at (64.0, -40.0)
- added LED_RGB_25: LED_RGB_5050-6, LED_RGB_5050-6, F.Cu at (77.3, -40.0)
- added LED_RGB_26: LED_RGB_5050-6, LED_RGB_5050-6, F.Cu at (90.7, -40.0)
- added LED_RGB_27: LED_RGB_5050-6, LED_RGB_5050-6, F.Cu at (104.0, -40.0)
- added LED_RGB_28: LED_RGB_5050-6, LED_RGB_5050-6, F.Cu at (117.3, -40.0)
- added LED_RGB_29: LED_RGB_5050-6, LED_RGB_5050-6, F.Cu at (130.7, -40.0)
- added LED_RGB_3: LED_RGB_5050-6, LED_RGB_5050-6, F.Cu at (1.00, -40.0)
- added LED_RGB_30: LED_RGB_5050-6, LED_RGB_5050-6, F.Cu at (143.0, -39.0)
- added LED_RGB_31: LED_RGB_5050-6, LED_RGB_5050-6, F.Cu at (143.0, -25.7)
- added LED_RGB_32: LED_RGB_5050-6, LED_RGB_5050-6, F.Cu at (143.0, -12.3)
- added LED_RGB_33: LED_RGB_5050-6, LED_RGB_5050-6, F.Cu at (143.0, 1.00)
- added LED_RGB_34: LED_RGB_5050-6, LED_RGB_5050-6, F.Cu at (143.0, 14.3)
- added LED_RGB_35: LED_RGB_5050-6, LED_RGB_5050-6, F.Cu at (143.0, 27.7)
- added LED_RGB_36: LED_RGB_5050-6, LED_RGB_5050-6, F.Cu at (142.0, 40.0)
- added LED_RGB_37: LED_RGB_5050-6, LED_RGB_5050-6, F.Cu at (128.7, 40.0)
- added LED_RGB_38: LED_RGB_5050-6, LED_RGB_5050-6, F.Cu at (115.3, 40.0)
- added LED_RGB_39: LED_RGB_5050-6, LED_RGB_5050-6, F.Cu at (102.0, 40.0)
- added LED_RGB_4: LED_RGB_5050-6, LED_RGB_5050-6, F.Cu at (14.3, -40.0)
- added LED_RGB_40: LED_RGB_5050-6, LED_RGB_5050-6, F.Cu at (88.7, 40.0)
- added LED_RGB_41: LED_RGB_5050-6, LED_RGB_5050-6, F.Cu at (75.3, 40.0)
- added LED_RGB_42: LED_RGB_5050-6, LED_RGB_5050-6, F.Cu at (63.0, 39.0)
- added LED_RGB_43: LED_RGB_5050-6, LED_RGB_5050-6, F.Cu at (63.0, 25.7)
- added LED_RGB_44: LED_RGB_5050-6, LED_RGB_5050-6, F.Cu at (63.0, 12.3)
- added LED_RGB_45: LED_RGB_5050-6, LED_RGB_5050-6, F.Cu at (63.0, -1.00)
- added LED_RGB_46: LED_RGB_5050-6, LED_RGB_5050-6, F.Cu at (63.0, -14.3)
- added LED_RGB_47: LED_RGB_5050-6, LED_RGB_5050-6, F.Cu at (63.0, -27.7)
- added LED_RGB_48: LED_RGB_5050-6, LED_RGB_5050-6, F.Cu at (-39.0, 63.0)
- added LED_RGB_49: LED_RGB_5050-6, LED_RGB_5050-6, F.Cu at (-25.7, 63.0)
- added LED_RGB_5: LED_RGB_5050-6, LED_RGB_5050-6, F.Cu at (27.7, -40.0)
- added LED_RGB_50: LED_RGB_5050-6, LED_RGB_5050-6, F.Cu at (-12.3, 63.0)
- added LED_RGB_51: LED_RGB_5050-6, LED_RGB_5050-6, F.Cu at (1.00, 63.0)
- added LED_RGB_52: LED_RGB_5050-6, LED_RGB_5050-6, F.Cu at (14.3, 63.0)
- added LED_RGB_53: LED_RGB_5050-6, LED_RGB_5050-6, F.Cu at (27.7, 63.0)
- added LED_RGB_54: LED_RGB_5050-6, LED_RGB_5050-6, F.Cu at (40.0, 64.0)
- added LED_RGB_55: LED_RGB_5050-6, LED_RGB_5050-6, F.Cu at (40.0, 77.3)
- added LED_RGB_56: LED_RGB_5050-6, LED_RGB_5050-6, F.Cu at (40.0, 90.7)
- added LED_RGB_57: LED_RGB_5050-6, LED_RGB_5050-6, F.Cu at (40.0, 104.0)
- added LED_RGB_58: LED_RGB_5050-6, LED_RGB_5050-6, F.Cu at (40.0, 117.3)
- added LED_RGB_59: LED_RGB_5050-6, LED_RGB_5050-6, F.Cu at (40.0, 130.7)
- added LED_RGB_6: LED_RGB_5050-6, LED_RGB_5050-6, F.Cu at (40.0, -39.0)
- added LED_RGB_60: LED_RGB_5050-6, LED_RGB_5050-6, F.Cu at (39.0, 143.0)
- added LED_RGB_61: LED_RGB_5050-6, LED_RGB_5050-6, F.Cu at (25.7, 143.0)
- added LED_RGB_62: LED_RGB_5050-6, LED_RGB_5050-6, F.Cu at (12.3, 143.0)
- added LED_RGB_63: LED_RGB_5050-6, LED_RGB_5050-6, F.Cu at (-1.00, 143.0)
- added LED_RGB_64: LED_RGB_5050-6, LED_RGB_5050-6, F.Cu at (-14.3, 143.0)
- added LED_RGB_65: LED_RGB_5050-6, LED_RGB_5050-6, F.Cu at (-27.7, 143.0)
- added LED_RGB_66: LED_RGB_5050-6, LED_RGB_5050-6, F.Cu at (-40.0, 142.0)
- added LED_RGB_67: LED_RGB_5050-6, LED_RGB_5050-6, F.Cu at (-40.0, 128.7)
- added LED_RGB_68: LED_RGB_5050-6, LED_RGB_5050-6, F.Cu at (-40.0, 115.3)
- added LED_RGB_69: LED_RGB_5050-6, LED_RGB_5050-6, F.Cu at (-40.0, 102.0)
- added LED_RGB_7: LED_RGB_5050-6, LED_RGB_5050-6, F.Cu at (40.0, -25.7)
- added LED_RGB_70: LED_RGB_5050-6, LED_RGB_5050-6, F.Cu at (-40.0, 88.7)
- added LED_RGB_71: LED_RGB_5050-6, LED_RGB_5050-6, F.Cu at (-40.0, 75.3)
- added LED_RGB_72: LED_RGB_5050-6, LED_RGB_5050-6, F.Cu at (64.0, 63.0)
- added LED_RGB_73: LED_RGB_5050-6, LED_RGB_5050-6, F.Cu at (77.3, 63.0)
- added LED_RGB_74: LED_RGB_5050-6, LED_RGB_5050-6, F.Cu at (90.7, 63.0)
- added LED_RGB_75: LED_RGB_5050-6, LED_RGB_5050-6, F.Cu at (104.0, 63.0)
- added LED_RGB_76: LED_RGB_5050-6, LED_RGB_5050-6, F.Cu at (117.3, 63.0)
- added LED_RGB_77: LED_RGB_5050-6, LED_RGB_5050-6, F.Cu at (130.7, 63.0)
- added LED_RGB_78: LED_RGB_5050-6, LED_RGB_5050-6, F.Cu at (143.0, 64.0)
- added LED_RGB_79: LED_RGB_5050-6, LED_RGB_5050-6, F.Cu at (143.0, 77.3)
- added LED_RGB_8: LED_RGB_5050-6, LED_RGB_5050-6, F.Cu at (40.0, -12.3)
- added LED_RGB_80: LED_RGB_5050-6, LED_RGB_5050-6, F.Cu at (143.0, 90.7)
- added LED_RGB_81: LED_RGB_5050-6, LED_RGB_5050-6, F.Cu at (143.0, 104.0)
- added LED_RGB_82: LED_RGB_5050-6, LED_RGB_5050-6, F.Cu at (143.0, 117.3)
- added LED_RGB_83: LED_RGB_5050-6, LED_RGB_5050-6, F.Cu at (143.0, 130.7)
- added LED_RGB_84: LED_RGB_5050-6, LED_RGB_5050-6, F.Cu at (142.0, 143.0)
- added LED_RGB_85: LED_RGB_5050-6, LED_RGB_5050-6, F.Cu at (128.7, 143.0)
- added LED_RGB_86: LED_RGB_5050-6, LED_RGB_5050-6, F.Cu at (115.3, 143.0)
- added LED_RGB_87: LED_RGB_5050-6, LED_RGB_5050-6, F.Cu at (102.0, 143.0)
- added LED_RGB_88: LED_RGB_5050-6, LED_RGB_5050-6, F.Cu at (88.7, 143.0)
- added LED_RGB_89: LED_RGB_5050-6, LED_RGB_5050-6, F.Cu at (75.3, 143.0)
- added LED_RGB_9: LED_RGB_5050-6, LED_RGB_5050-6, F.Cu at (40.0, 1.00)
- added LED_RGB_90: LED_RGB_5050-6, LED_RGB_5050-6, F.Cu at (63.0, 142.0)
- added LED_RGB_91: LED_RGB_5050-6, LED_RGB_5050-6, F.Cu at (63.0, 128.7)
- added LED_RGB_92: LED_RGB_5050-6, LED_RGB_5050-6, F.Cu at (63.0, 115.3)
- added LED_RGB_93: LED_RGB_5050-6, LED_RGB_5050-6, F.Cu at (63.0, 102.0)
- added LED_RGB_94: LED_RGB_5050-6, LED_RGB_5050-6, F.Cu at (63.0, 88.7)
- added LED_RGB_95: LED_RGB_5050-6, LED_RGB_5050-6, F.Cu at (63.0, 75.3)
- added LED_W2_0: LED_RGB_5050-6, LED_RGB_5050-6, F.Cu at (-6.50, -7.50)
- added LED_W2_1: LED_RGB_5050-6, LED_RGB_5050-6, F.Cu at (7.50, -6.50)
- added LED_W2_10: LED_RGB_5050-6, LED_RGB_5050-6, F.Cu at (6.50, 110.5)
- added LED_W2_11: LED_RGB_5050-6, LED_RGB_5050-6, F.Cu at (-7.50, 109.5)
- added LED_W2_12: LED_RGB_5050-6, LED_RGB_5050-6, F.Cu at (96.5, 95.5)
- added LED_W2_13: LED_RGB_5050-6, LED_RGB_5050-6, F.Cu at (110.5, 96.5)
- added LED_W2_14: LED_RGB_5050-6, LED_RGB_5050-6, F.Cu at (109.5, 110.5)
- added LED_W2_15: LED_RGB_5050-6, LED_RGB_5050-6, F.Cu at (95.5, 109.5)
- added LED_W2_2: LED_RGB_5050-6, LED_RGB_5050-6, F.Cu at (6.50, 7.50)
- added LED_W2_3: LED_RGB_5050-6, LED_RGB_5050-6, F.Cu at (-7.50, 6.50)
- added LED_W2_4: LED_RGB_5050-6, LED_RGB_5050-6, F.Cu at (96.5, -7.50)
- added LED_W2_5: LED_RGB_5050-6, LED_RGB_5050-6, F.Cu at (110.5, -6.50)
- added LED_W2_6: LED_RGB_5050-6, LED_RGB_5050-6, F.Cu at (109.5, 7.50)
- added LED_W2_7: LED_RGB_5050-6, LED_RGB_5050-6, F.Cu at (95.5, 6.50)
- added LED_W2_8: LED_RGB_5050-6, LED_RGB_5050-6, F.Cu at (-6.50, 95.5)
- added LED_W2_9: LED_RGB_5050-6, LED_RGB_5050-6, F.Cu at (7.50, 96.5)
- added LED_W_0: LED_RGB_5050-6, LED_RGB_5050-6, F.Cu at (-19.0, -20.0)
- added LED_W_1: LED_RGB_5050-6, LED_RGB_5050-6, F.Cu at (-5.67, -20.0)
- added LED_W_10: LED_RGB_5050-6, LED_RGB_5050-6, F.Cu at (-20.0, 5.67)
- added LED_W_11: LED_RGB_5050-6, LED_RGB_5050-6, F.Cu at (-20.0, -7.67)
- added LED_W_12: LED_RGB_5050-6, LED_RGB_5050-6, F.Cu at (84.0, -20.0)
- added LED_W_13: LED_RGB_5050-6, LED_RGB_5050-6, F.Cu at (97.3, -20.0)
- added LED_W_14: LED_RGB_5050-6, LED_RGB_5050-6, F.Cu at (110.7, -20.0)
- added LED_W_15: LED_RGB_5050-6, LED_RGB_5050-6, F.Cu at (123.0, -19.0)
- added LED_W_16: LED_RGB_5050-6, LED_RGB_5050-6, F.Cu at (123.0, -5.67)
- added LED_W_17: LED_RGB_5050-6, LED_RGB_5050-6, F.Cu at (123.0, 7.67)
- added LED_W_18: LED_RGB_5050-6, LED_RGB_5050-6, F.Cu at (122.0, 20.0)
- added LED_W_19: LED_RGB_5050-6, LED_RGB_5050-6, F.Cu at (108.7, 20.0)
- added LED_W_2: LED_RGB_5050-6, LED_RGB_5050-6, F.Cu at (7.67, -20.0)
- added LED_W_20: LED_RGB_5050-6, LED_RGB_5050-6, F.Cu at (95.3, 20.0)
- added LED_W_21: LED_RGB_5050-6, LED_RGB_5050-6, F.Cu at (83.0, 19.0)
- added LED_W_22: LED_RGB_5050-6, LED_RGB_5050-6, F.Cu at (83.0, 5.67)
- added LED_W_23: LED_RGB_5050-6, LED_RGB_5050-6, F.Cu at (83.0, -7.67)
- added LED_W_24: LED_RGB_5050-6, LED_RGB_5050-6, F.Cu at (-19.0, 83.0)
- added LED_W_25: LED_RGB_5050-6, LED_RGB_5050-6, F.Cu at (-5.67, 83.0)
- added LED_W_26: LED_RGB_5050-6, LED_RGB_5050-6, F.Cu at (7.67, 83.0)
- added LED_W_27: LED_RGB_5050-6, LED_RGB_5050-6, F.Cu at (20.0, 84.0)
- added LED_W_28: LED_RGB_5050-6, LED_RGB_5050-6, F.Cu at (20.0, 97.3)
- added LED_W_29: LED_RGB_5050-6, LED_RGB_5050-6, F.Cu at (20.0, 110.7)
- added LED_W_3: LED_RGB_5050-6, LED_RGB_5050-6, F.Cu at (20.0, -19.0)
- added LED_W_30: LED_RGB_5050-6, LED_RGB_5050-6, F.Cu at (19.0, 123.0)
- added LED_W_31: LED_RGB_5050-6, LED_RGB_5050-6, F.Cu at (5.67, 123.0)
- added LED_W_32: LED_RGB_5050-6, LED_RGB_5050-6, F.Cu at (-7.67, 123.0)
- added LED_W_33: LED_RGB_5050-6, LED_RGB_5050-6, F.Cu at (-20.0, 122.0)
- added LED_W_34: LED_RGB_5050-6, LED_RGB_5050-6, F.Cu at (-20.0, 108.7)
- added LED_W_35: LED_RGB_5050-6, LED_RGB_5050-6, F.Cu at (-20.0, 95.3)
- added LED_W_36: LED_RGB_5050-6, LED_RGB_5050-6, F.Cu at (84.0, 83.0)
- added LED_W_37: LED_RGB_5050-6, LED_RGB_5050-6, F.Cu at (97.3, 83.0)
- added LED_W_38: LED_RGB_5050-6, LED_RGB_5050-6, F.Cu at (110.7, 83.0)
- added LED_W_39: LED_RGB_5050-6, LED_RGB_5050-6, F.Cu at (123.0, 84.0)
- added LED_W_4: LED_RGB_5050-6, LED_RGB_5050-6, F.Cu at (20.0, -5.67)
- added LED_W_40: LED_RGB_5050-6, LED_RGB_5050-6, F.Cu at (123.0, 97.3)
- added LED_W_41: LED_RGB_5050-6, LED_RGB_5050-6, F.Cu at (123.0, 110.7)
- added LED_W_42: LED_RGB_5050-6, LED_RGB_5050-6, F.Cu at (122.0, 123.0)
- added LED_W_43: LED_RGB_5050-6, LED_RGB_5050-6, F.Cu at (108.7, 123.0)
- added LED_W_44: LED_RGB_5050-6, LED_RGB_5050-6, F.Cu at (95.3, 123.0)
- added LED_W_45: LED_RGB_5050-6, LED_RGB_5050-6, F.Cu at (83.0, 122.0)
- added LED_W_46: LED_RGB_5050-6, LED_RGB_5050-6, F.Cu at (83.0, 108.7)
- added LED_W_47: LED_RGB_5050-6, LED_RGB_5050-6, F.Cu at (83.0, 95.3)
- added LED_W_5: LED_RGB_5050-6, LED_RGB_5050-6, F.Cu at (20.0, 7.67)
- added LED_W_6: LED_RGB_5050-6, LED_RGB_5050-6, F.Cu at (19.0, 20.0)
- added LED_W_7: LED_RGB_5050-6, LED_RGB_5050-6, F.Cu at (5.67, 20.0)
- added LED_W_8: LED_RGB_5050-6, LED_RGB_5050-6, F.Cu at (-7.67, 20.0)
- added LED_W_9: LED_RGB_5050-6, LED_RGB_5050-6, F.Cu at (-20.0, 19.0)
- added R_0_0_RGB: R_0603_1608Metric, R_0603_1608Metric, F.Cu at (-45.0, -40.0)
- added R_0_0_RGB1: R_0603_1608Metric, R_0603_1608Metric, F.Cu at (58.0, -40.0)
- added R_0_0_RGB2: R_0603_1608Metric, R_0603_1608Metric, F.Cu at (-35.0, -30.0)
- added R_0_0_RGB3: R_0603_1608Metric, R_0603_1608Metric, F.Cu at (68.0, -30.0)
- added R_0_0_RGB4: R_0603_1608Metric, R_0603_1608Metric, F.Cu at (-45.0, 63.0)
- added R_0_0_RGB5: R_0603_1608Metric, R_0603_1608Metric, F.Cu at (-35.0, 73.0)
- added R_0_0_RGB6: R_0603_1608Metric, R_0603_1608Metric, F.Cu at (58.0, 63.0)
- added R_0_0_RGB7: R_0603_1608Metric, R_0603_1608Metric, F.Cu at (68.0, 73.0)
- added R_0_0_W: R_0603_1608Metric, R_0603_1608Metric, F.Cu at (-25.0, -20.0)
- added R_0_0_W1: R_0603_1608Metric, R_0603_1608Metric, F.Cu at (78.0, -20.0)
- added R_0_0_W2: R_0603_1608Metric, R_0603_1608Metric, F.Cu at (-12.5, -7.50)
- added R_0_0_W3: R_0603_1608Metric, R_0603_1608Metric, F.Cu at (90.5, -7.50)
- added R_0_0_W4: R_0603_1608Metric, R_0603_1608Metric, F.Cu at (-25.0, 83.0)
- added R_0_0_W5: R_0603_1608Metric, R_0603_1608Metric, F.Cu at (-12.5, 95.5)
- added R_0_0_W6: R_0603_1608Metric, R_0603_1608Metric, F.Cu at (78.0, 83.0)
- added R_0_0_W7: R_0603_1608Metric, R_0603_1608Metric, F.Cu at (90.5, 95.5)
- added R_0_1_RGB: R_0603_1608Metric, R_0603_1608Metric, F.Cu at (-45.0, -42.0)
- added R_0_1_RGB1: R_0603_1608Metric, R_0603_1608Metric, F.Cu at (58.0, -42.0)
- added R_0_1_RGB2: R_0603_1608Metric, R_0603_1608Metric, F.Cu at (-35.0, -32.0)
- added R_0_1_RGB3: R_0603_1608Metric, R_0603_1608Metric, F.Cu at (68.0, -32.0)
- added R_0_1_RGB4: R_0603_1608Metric, R_0603_1608Metric, F.Cu at (-45.0, 61.0)
- added R_0_1_RGB5: R_0603_1608Metric, R_0603_1608Metric, F.Cu at (-35.0, 71.0)
- added R_0_1_RGB6: R_0603_1608Metric, R_0603_1608Metric, F.Cu at (58.0, 61.0)
- added R_0_1_RGB7: R_0603_1608Metric, R_0603_1608Metric, F.Cu at (68.0, 71.0)
- added R_0_2_RGB: R_0603_1608Metric, R_0603_1608Metric, F.Cu at (-45.0, -38.0)
- added R_0_2_RGB1: R_0603_1608Metric, R_0603_1608Metric, F.Cu at (58.0, -38.0)
- added R_0_2_RGB2: R_0603_1608Metric, R_0603_1608Metric, F.Cu at (-35.0, -28.0)
- added R_0_2_RGB3: R_0603_1608Metric, R_0603_1608Metric, F.Cu at (68.0, -28.0)
- added R_0_2_RGB4: R_0603_1608Metric, R_0603_1608Metric, F.Cu at (-45.0, 65.0)
- added R_0_2_RGB5: R_0603_1608Metric, R_0603_1608Metric, F.Cu at (-35.0, 75.0)
- added R_0_2_RGB6: R_0603_1608Metric, R_0603_1608Metric, F.Cu at (58.0, 65.0)
- added R_0_2_RGB7: R_0603_1608Metric, R_0603_1608Metric, F.Cu at (68.0, 75.0)
- added R_10_0_W: R_0603_1608Metric, R_0603_1608Metric, F.Cu at (-20.0, 11.7)
- added R_10_0_W1: R_0603_1608Metric, R_0603_1608Metric, F.Cu at (83.0, 11.7)
- added R_10_0_W2: R_0603_1608Metric, R_0603_1608Metric, F.Cu at (-20.0, 114.7)
- added R_10_0_W3: R_0603_1608Metric, R_0603_1608Metric, F.Cu at (83.0, 114.7)
- added R_12_0_RGB: R_0603_1608Metric, R_0603_1608Metric, F.Cu at (45.0, 40.0)
- added R_12_0_RGB1: R_0603_1608Metric, R_0603_1608Metric, F.Cu at (148.0, 40.0)
- added R_12_0_RGB2: R_0603_1608Metric, R_0603_1608Metric, F.Cu at (45.0, 143.0)
- added R_12_0_RGB3: R_0603_1608Metric, R_0603_1608Metric, F.Cu at (148.0, 143.0)
- added R_12_1_RGB: R_0603_1608Metric, R_0603_1608Metric, F.Cu at (45.0, 42.0)
- added R_12_1_RGB1: R_0603_1608Metric, R_0603_1608Metric, F.Cu at (148.0, 42.0)
- added R_12_1_RGB2: R_0603_1608Metric, R_0603_1608Metric, F.Cu at (45.0, 145.0)
- added R_12_1_RGB3: R_0603_1608Metric, R_0603_1608Metric, F.Cu at (148.0, 145.0)
- added R_12_2_RGB: R_0603_1608Metric, R_0603_1608Metric, F.Cu at (45.0, 38.0)
- added R_12_2_RGB1: R_0603_1608Metric, R_0603_1608Metric, F.Cu at (148.0, 38.0)
- added R_12_2_RGB2: R_0603_1608Metric, R_0603_1608Metric, F.Cu at (45.0, 141.0)
- added R_12_2_RGB3: R_0603_1608Metric, R_0603_1608Metric, F.Cu at (148.0, 141.0)
- added R_15_0_RGB: R_0603_1608Metric, R_0603_1608Metric, F.Cu at (5.00, 40.0)
- added R_15_0_RGB1: R_0603_1608Metric, R_0603_1608Metric, F.Cu at (108.0, 40.0)
- added R_15_0_RGB2: R_0603_1608Metric, R_0603_1608Metric, F.Cu at (5.00, 143.0)
- added R_15_0_RGB3: R_0603_1608Metric, R_0603_1608Metric, F.Cu at (108.0, 143.0)
- added R_15_1_RGB: R_0603_1608Metric, R_0603_1608Metric, F.Cu at (5.00, 42.0)
- added R_15_1_RGB1: R_0603_1608Metric, R_0603_1608Metric, F.Cu at (108.0, 42.0)
- added R_15_1_RGB2: R_0603_1608Metric, R_0603_1608Metric, F.Cu at (5.00, 145.0)
- added R_15_1_RGB3: R_0603_1608Metric, R_0603_1608Metric, F.Cu at (108.0, 145.0)
- added R_15_2_RGB: R_0603_1608Metric, R_0603_1608Metric, F.Cu at (5.00, 38.0)
- added R_15_2_RGB1: R_0603_1608Metric, R_0603_1608Metric, F.Cu at (108.0, 38.0)
- added R_15_2_RGB2: R_0603_1608Metric, R_0603_1608Metric, F.Cu at (5.00, 141.0)
- added R_15_2_RGB3: R_0603_1608Metric, R_0603_1608Metric, F.Cu at (108.0, 141.0)
- added R_18_0_RGB: R_0603_1608Metric, R_0603_1608Metric, F.Cu at (-40.0, 45.0)
- added R_18_0_RGB1: R_0603_1608Metric, R_0603_1608Metric, F.Cu at (63.0, 45.0)
- added R_18_0_RGB2: R_0603_1608Metric, R_0603_1608Metric, F.Cu at (-40.0, 148.0)
- added R_18_0_RGB3: R_0603_1608Metric, R_0603_1608Metric, F.Cu at (63.0, 148.0)
- added R_18_1_RGB: R_0603_1608Metric, R_0603_1608Metric, F.Cu at (-42.0, 45.0)
- added R_18_1_RGB1: R_0603_1608Metric, R_0603_1608Metric, F.Cu at (61.0, 45.0)
- added R_18_1_RGB2: R_0603_1608Metric, R_0603_1608Metric, F.Cu at (-42.0, 148.0)
- added R_18_1_RGB3: R_0603_1608Metric, R_0603_1608Metric, F.Cu at (61.0, 148.0)
- added R_18_2_RGB: R_0603_1608Metric, R_0603_1608Metric, F.Cu at (-38.0, 45.0)
- added R_18_2_RGB1: R_0603_1608Metric, R_0603_1608Metric, F.Cu at (65.0, 45.0)
- added R_18_2_RGB2: R_0603_1608Metric, R_0603_1608Metric, F.Cu at (-38.0, 148.0)
- added R_18_2_RGB3: R_0603_1608Metric, R_0603_1608Metric, F.Cu at (65.0, 148.0)
- added R_21_0_RGB: R_0603_1608Metric, R_0603_1608Metric, F.Cu at (-40.0, 5.00)
- added R_21_0_RGB1: R_0603_1608Metric, R_0603_1608Metric, F.Cu at (63.0, 5.00)
- added R_21_0_RGB2: R_0603_1608Metric, R_0603_1608Metric, F.Cu at (-40.0, 108.0)
- added R_21_0_RGB3: R_0603_1608Metric, R_0603_1608Metric, F.Cu at (63.0, 108.0)
- added R_21_1_RGB: R_0603_1608Metric, R_0603_1608Metric, F.Cu at (-42.0, 5.00)
- added R_21_1_RGB1: R_0603_1608Metric, R_0603_1608Metric, F.Cu at (61.0, 5.00)
- added R_21_1_RGB2: R_0603_1608Metric, R_0603_1608Metric, F.Cu at (-42.0, 108.0)
- added R_21_1_RGB3: R_0603_1608Metric, R_0603_1608Metric, F.Cu at (61.0, 108.0)
- added R_21_2_RGB: R_0603_1608Metric, R_0603_1608Metric, F.Cu at (-38.0, 5.00)
- added R_21_2_RGB1: R_0603_1608Metric, R_0603_1608Metric, F.Cu at (65.0, 5.00)
- added R_21_2_RGB2: R_0603_1608Metric, R_0603_1608Metric, F.Cu at (-38.0, 108.0)
- added R_21_2_RGB3: R_0603_1608Metric, R_0603_1608Metric, F.Cu at (65.0, 108.0)
- added R_2_0_W: R_0603_1608Metric, R_0603_1608Metric, F.Cu at (1.67, -20.0)
- added R_2_0_W1: R_0603_1608Metric, R_0603_1608Metric, F.Cu at (104.7, -20.0)
- added R_2_0_W2: R_0603_1608Metric, R_0603_1608Metric, F.Cu at (12.5, 7.50)
- added R_2_0_W3: R_0603_1608Metric, R_0603_1608Metric, F.Cu at (115.5, 7.50)
- added R_2_0_W4: R_0603_1608Metric, R_0603_1608Metric, F.Cu at (1.67, 83.0)
- added R_2_0_W5: R_0603_1608Metric, R_0603_1608Metric, F.Cu at (12.5, 110.5)
- added R_2_0_W6: R_0603_1608Metric, R_0603_1608Metric, F.Cu at (104.7, 83.0)
- added R_2_0_W7: R_0603_1608Metric, R_0603_1608Metric, F.Cu at (115.5, 110.5)
- added R_3_0_RGB: R_0603_1608Metric, R_0603_1608Metric, F.Cu at (-5.00, -40.0)
- added R_3_0_RGB1: R_0603_1608Metric, R_0603_1608Metric, F.Cu at (98.0, -40.0)
- added R_3_0_RGB2: R_0603_1608Metric, R_0603_1608Metric, F.Cu at (30.0, -35.0)
- added R_3_0_RGB3: R_0603_1608Metric, R_0603_1608Metric, F.Cu at (133.0, -35.0)
- added R_3_0_RGB4: R_0603_1608Metric, R_0603_1608Metric, F.Cu at (-5.00, 63.0)
- added R_3_0_RGB5: R_0603_1608Metric, R_0603_1608Metric, F.Cu at (30.0, 68.0)
- added R_3_0_RGB6: R_0603_1608Metric, R_0603_1608Metric, F.Cu at (98.0, 63.0)
- added R_3_0_RGB7: R_0603_1608Metric, R_0603_1608Metric, F.Cu at (133.0, 68.0)
- added R_3_1_RGB: R_0603_1608Metric, R_0603_1608Metric, F.Cu at (-5.00, -42.0)
- added R_3_1_RGB1: R_0603_1608Metric, R_0603_1608Metric, F.Cu at (98.0, -42.0)
- added R_3_1_RGB2: R_0603_1608Metric, R_0603_1608Metric, F.Cu at (32.0, -35.0)
- added R_3_1_RGB3: R_0603_1608Metric, R_0603_1608Metric, F.Cu at (135.0, -35.0)
- added R_3_1_RGB4: R_0603_1608Metric, R_0603_1608Metric, F.Cu at (-5.00, 61.0)
- added R_3_1_RGB5: R_0603_1608Metric, R_0603_1608Metric, F.Cu at (32.0, 68.0)
- added R_3_1_RGB6: R_0603_1608Metric, R_0603_1608Metric, F.Cu at (98.0, 61.0)
- added R_3_1_RGB7: R_0603_1608Metric, R_0603_1608Metric, F.Cu at (135.0, 68.0)
- added R_3_2_RGB: R_0603_1608Metric, R_0603_1608Metric, F.Cu at (-5.00, -38.0)
- added R_3_2_RGB1: R_0603_1608Metric, R_0603_1608Metric, F.Cu at (98.0, -38.0)
- added R_3_2_RGB2: R_0603_1608Metric, R_0603_1608Metric, F.Cu at (28.0, -35.0)
- added R_3_2_RGB3: R_0603_1608Metric, R_0603_1608Metric, F.Cu at (131.0, -35.0)
- added R_3_2_RGB4: R_0603_1608Metric, R_0603_1608Metric, F.Cu at (-5.00, 65.0)
- added R_3_2_RGB5: R_0603_1608Metric, R_0603_1608Metric, F.Cu at (28.0, 68.0)
- added R_3_2_RGB6: R_0603_1608Metric, R_0603_1608Metric, F.Cu at (98.0, 65.0)
- added R_3_2_RGB7: R_0603_1608Metric, R_0603_1608Metric, F.Cu at (131.0, 68.0)
- added R_4_0_W: R_0603_1608Metric, R_0603_1608Metric, F.Cu at (20.0, -11.7)
- added R_4_0_W1: R_0603_1608Metric, R_0603_1608Metric, F.Cu at (123.0, -11.7)
- added R_4_0_W2: R_0603_1608Metric, R_0603_1608Metric, F.Cu at (20.0, 91.3)
- added R_4_0_W3: R_0603_1608Metric, R_0603_1608Metric, F.Cu at (123.0, 91.3)
- added R_6_0_RGB: R_0603_1608Metric, R_0603_1608Metric, F.Cu at (40.0, -45.0)
- added R_6_0_RGB1: R_0603_1608Metric, R_0603_1608Metric, F.Cu at (143.0, -45.0)
- added R_6_0_RGB2: R_0603_1608Metric, R_0603_1608Metric, F.Cu at (35.0, 30.0)
- added R_6_0_RGB3: R_0603_1608Metric, R_0603_1608Metric, F.Cu at (138.0, 30.0)
- added R_6_0_RGB4: R_0603_1608Metric, R_0603_1608Metric, F.Cu at (40.0, 58.0)
- added R_6_0_RGB5: R_0603_1608Metric, R_0603_1608Metric, F.Cu at (35.0, 133.0)
- added R_6_0_RGB6: R_0603_1608Metric, R_0603_1608Metric, F.Cu at (143.0, 58.0)
- added R_6_0_RGB7: R_0603_1608Metric, R_0603_1608Metric, F.Cu at (138.0, 133.0)
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Routing:
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Other:
- board outline added: 203 x 203 mm
