File: hardware/TIYCS_main/TIYCS_main.kicad_sch (KiCad schematic)
At the start: 48 parts, among them J1 USB4105-GF-A, J2 12vPWM, J3 WS2812B, J4 UART, J5 ExtSensor, J6 Terminal, J7 Barrel_Jack_Switch, J8 pinHeaders, Q1 NCE4060K, Q2 NCE4060K, Q3 2N7002, Q4 NCE4060K, Q5 NCE4060K, SW1 RST, SW2 BOOT, SW3 BTN, U1 ESP32-WROOM-32U, U2 CH340N, U3 XL-1509-3.3E1

Commit message: Added XT60 conn to battery board
Parts:
- SW3: footprint Switches:TACTILE_SWITCH_SMD_6.0X3.5MM -> Button_Switch_SMD:SW_SPST_CK_RS282G05A3
Changed lines of the file:
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@@
     (property "Reference" "SW3" (id 0) (at 108.585 133.4475 0))
     (property "Value" "BTN" (id 1) (at 108.585 136.2226 0))
-    (property "Footprint" "Switches:TACTILE_SWITCH_SMD_6.0X3.5MM" (id 2) (at 108.585 142.875 0)
+    (property "Footprint" "Button_Switch_SMD:SW_SPST_CK_RS282G05A3" (id 2) (at 108.585 142.875 0)
       (effects (font (size 1.27 1.27)) hide)
     )
@@
     )
     (path "/d13e8b6d-8b82-4ae1-a8ab-4cc22756669a"
-      (reference "SW3") (unit 1) (value "BTN") (footprint "Switches:TACTILE_SWITCH_SMD_6.0X3.5MM")
+      (reference "SW3") (unit 1) (value "BTN") (footprint "Button_Switch_SMD:SW_SPST_CK_RS282G05A3")
     )
     (path "/f3889d7e-5766-4016-abdb-86011b33eeb0"

Commit message: Updated README
Parts:
- added R4: 10K, Resistor_SMD:R_0603_1608Metric, symbol Device:R
Connections:
- net V_SENSE: now also R4.1; no longer Q3.1 (G), R8.2
- new net: Q3.1 (G), R4.2, R8.2
Other:
- moved on the sheet: Q3, R11, R8
Changed lines of the file:
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@@
   (junction (at 142.875 48.26) (diameter 0) (color 0 0 0 0)
   )
-  (junction (at 226.695 146.05) (diameter 1.016) (color 0 0 0 0)
+  (junction (at 238.125 146.05) (diameter 1.016) (color 0 0 0 0)
   )
   (junction (at 247.65 62.865) (diameter 0) (color 0 0 0 0)
@@
     (stroke (width 0) (type solid) (color 0 0 0 0))
   )
-  (wire (pts (xy 223.52 146.05) (xy 226.695 146.05))
+  (wire (pts (xy 234.95 146.05) (xy 238.125 146.05))
     (stroke (width 0) (type solid) (color 0 0 0 0))
   )
@@
     )
   )
-  (global_label "SENSE_PIN" (shape input) (at 234.315 151.13 270) (fields_autoplaced)
-    (effects (font (size 1.27 1.27)) (justify right))
-    (property "Intersheet References" "${INTERSHEET_REFS}" (id 0) (at 234.2356 163.7636 90)
+  (global_label "SENSE_PIN" (shape input) (at 245.745 151.13 270) (fields_autoplaced)
+    (effects (font (size 1.27 1.27)) (justify right))
+    (property "Intersheet References" "${INTERSHEET_REFS}" (id 0) (at 245.6656 163.7636 90)
       (effects (font (size 1.27 1.27)) (justify right) hide)
     )
@@
     )
   )
-  (global_label "V_SENSE" (shape input) (at 223.52 146.05 180) (fields_autoplaced)
-    (effects (font (size 1.27 1.27)) (justify right))
-    (property "Intersheet References" "${INTERSHEET_REFS}" (id 0) (at 213.0031 145.9706 0)
+  (global_label "V_SENSE" (shape input) (at 227.33 146.05 180) (fields_autoplaced)
+    (effects (font (size 1.27 1.27)) (justify right))
+    (property "Intersheet References" "${INTERSHEET_REFS}" (id 0) (at 216.8131 145.9706 0)
       (effects (font (size 1.27 1.27)) (justify right) hide)
     )
@@
     (pin "3")
   )
-  (symbol (lib_id "power:+3.3V") (at 234.315 133.35 0) (unit 1)
-    (in_bom yes) (on_board yes) (fields_autoplaced)
-    (property "Reference" "#PWR0118" (id 0) (at 234.315 137.16 0)
-      (effects (font (size 1.27 1.27)) hide)
-    )
-    (property "Value" "+3.3V" (id 1) (at 234.315 129.8026 0))
-    (property "Footprint" "" (id 2) (at 234.315 133.35 0)
-      (effects (font (size 1.27 1.27)) hide)
-    )
-    (property "Datasheet" "" (id 3) (at 234.315 133.35 0)
+  (symbol (lib_id "power:+3.3V") (at 245.745 133.35 0) (unit 1)
+    (in_bom yes) (on_board yes) (fields_autoplaced)
+    (property "Reference" "#PWR0118" (id 0) (at 245.745 137.16 0)
+      (effects (font (size 1.27 1.27)) hide)
+    )
+    (property "Value" "+3.3V" (id 1) (at 245.745 129.8026 0))
+    (property "Footprint" "" (id 2) (at 245.745 133.35 0)
+      (effects (font (size 1.27 1.27)) hide)
+    )
+    (property "Datasheet" "" (id 3) (at 245.745 133.35 0)
       (effects (font (size 1.27 1.27)) hide)
     )
@@
     (pin "1")
   )
-  (symbol (lib_id "Device:R") (at 226.695 142.24 0) (unit 1)
-    (in_bom yes) (on_board yes) (fields_autoplaced)
-    (property "Reference" "R8" (id 0) (at 228.4731 141.4791 0)
-      (effects (font (size 1.27 1.27)) (justify left))
-    )
-    (property "Value" "100K" (id 1) (at 228.4731 143.7778 0)
-      (effects (font (size 1.27 1.27)) (justify left))
-    )
-    (property "Footprint" "Resistor_SMD:R_0402_1005Metric" (id 2) (at 224.917 142.24 90)
-      (effects (font (size 1.27 1.27)) hide)
-    )
-    (property "Datasheet" "~" (id 3) (at 226.695 142.24 0)
+  (symbol (lib_id "Device:R") (at 238.125 142.24 0) (unit 1)
+    (in_bom yes) (on_board yes) (fields_autoplaced)
+    (property "Reference" "R8" (id 0) (at 239.9031 141.4791 0)
+      (effects (font (size 1.27 1.27)) (justify left))
+    )
+    (property "Value" "100K" (id 1) (at 239.9031 143.7778 0)
+      (effects (font (size 1.27 1.27)) (justify left))
+    )
+    (property "Footprint" "Resistor_SMD:R_0402_1005Metric" (id 2) (at 236.347 142.24 90)
+      (effects (font (size 1.27 1.27)) hide)
+    )
+    (property "Datasheet" "~" (id 3) (at 238.125 142.24 0)
       (effects (font (size 1.27 1.27)) hide)
     )
@@
     (pin "1")
   )
-  (symbol (lib_id "power:GND") (at 226.695 138.43 180) (unit 1)
-    (in_bom yes) (on_board yes) (fields_autoplaced)
-    (property "Reference" "#PWR0119" (id 0) (at 226.695 132.08 0)
-      (effects (font (size 1.27 1.27)) hide)
-    )
-    (property "Value" "GND" (id 1) (at 226.695 134.8826 0))
-    (property "Footprint" "" (id 2) (at 226.695 138.43 0)
-      (effects (font (size 1.27 1.27)) hide)
-    )
-    (property "Datasheet" "" (id 3) (at 226.695 138.43 0)
+  (symbol (lib_id "power:GND") (at 238.125 138.43 180) (unit 1)
+    (in_bom yes) (on_board yes) (fields_autoplaced)
+    (property "Reference" "#PWR0119" (id 0) (at 238.125 132.08 0)
+      (effects (font (size 1.27 1.27)) hide)
+    )
+    (property "Value" "GND" (id 1) (at 238.125 134.8826 0))
+    (property "Footprint" "" (id 2) (at 238.125 138.43 0)
+      (effects (font (size 1.27 1.27)) hide)
+    )
+    (property "Datasheet" "" (id 3) (at 238.125 138.43 0)
       (effects (font (size 1.27 1.27)) hide)
     )
@@
     (pin "1")
   )
-  (symbol (lib_id "Device:R") (at 234.315 137.16 0) (unit 1)
-    (in_bom yes) (on_board yes) (fields_autoplaced)
-    (property "Reference" "R11" (id 0) (at 236.0931 136.3991 0)
-      (effects (font (size 1.27 1.27)) (justify left))
-    )
-    (property "Value" "100K" (id 1) (at 236.0931 138.6978 0)
-      (effects (font (size 1.27 1.27)) (justify left))
-    )
-    (property "Footprint" "Resistor_SMD:R_0402_1005Metric" (id 2) (at 232.537 137.16 90)
-      (effects (font (size 1.27 1.27)) hide)
-    )
-    (property "Datasheet" "~" (id 3) (at 234.315 137.16 0)
+  (symbol (lib_id "Device:R") (at 245.745 137.16 0) (unit 1)
+    (in_bom yes) (on_board yes) (fields_autoplaced)
+    (property "Reference" "R11" (id 0) (at 247.5231 136.3991 0)
+      (effects (font (size 1.27 1.27)) (justify left))
+    )
+    (property "Value" "100K" (id 1) (at 247.5231 138.6978 0)
+      (effects (font (size 1.27 1.27)) (justify left))
+    )
+    (property "Footprint" "Resistor_SMD:R_0402_1005Metric" (id 2) (at 243.967 137.16 90)
+      (effects (font (size 1.27 1.27)) hide)
+    )
+    (property "Datasheet" "~" (id 3) (at 245.745 137.16 0)
       (effects (font (size 1.27 1.27)) hide)
     )
@@
     (pin "2")
   )
-  (symbol (lib_id "Device:Q_NMOS_GSD") (at 231.775 146.05 0) (unit 1)
-    (in_bom yes) (on_board yes) (fields_autoplaced)
-    (property "Reference" "Q3" (id 0) (at 236.9821 145.2891 0)
-      (effects (font (size 1.27 1.27)) (justify left))
-    )
-    (property "Value" "2N7002" (id 1) (at 236.9821 147.5878 0)
-      (effects (font (size 1.27 1.27)) (justify left))
-    )
-    (property "Footprint" "Package_TO_SOT_SMD:SOT-23" (id 2) (at 236.855 143.51 0)
-      (effects (font (size 1.27 1.27)) hide)
-    )
-    (property "Datasheet" "~" (id 3) (at 231.775 146.05 0)
-      (effects (font (size 1.27 1.27)) hide)
-    )
-    (property "JLCPCB" "C8545 " (id 4) (at 231.775 146.05 0)
+  (symbol (lib_id "Device:Q_NMOS_GSD") (at 243.205 146.05 0) (unit 1)
+    (in_bom yes) (on_board yes) (fields_autoplaced)
+    (property "Reference" "Q3" (id 0) (at 248.4121 145.2891 0)
+      (effects (font (size 1.27 1.27)) (justify left))
+    )
+    (property "Value" "2N7002" (id 1) (at 248.4121 147.5878 0)
+      (effects (font (size 1.27 1.27)) (justify left))
+    )
+    (property "Footprint" "Package_TO_SOT_SMD:SOT-23" (id 2) (at 248.285 143.51 0)
+      (effects (font (size 1.27 1.27)) hide)
+    )
+    (property "Datasheet" "~" (id 3) (at 243.205 146.05 0)
+      (effects (font (size 1.27 1.27)) hide)
+    )
+    (property "JLCPCB" "C8545 " (id 4) (at 243.205 146.05 0)
       (effects (font (size 1.27 1.27)) hide)
     )
@@
     (pin "3")
   )
+  (symbol (lib_id "Device:R") (at 231.14 146.05 90) (unit 1)
+    (in_bom yes) (on_board yes) (fields_autoplaced)
+    (property "Reference" "R4" (id 0) (at 231.14 141.0675 90))
+    (property "Value" "10K" (id 1) (at 231.14 143.8426 90))
+    (property "Footprint" "Resistor_SMD:R_0603_1608Metric" (id 2) (at 231.14 147.828 90)
+      (effects (font (size 1.27 1.27)) hide)
+    )
+    (property "Datasheet" "~" (id 3) (at 231.14 146.05 0)
+      (effects (font (size 1.27 1.27)) hide)
+    )
+    (pin "1")
+    (pin "2")
+  )
   (symbol (lib_id "Device:C_Polarized") (at 196.85 52.07 0) (unit 1)
     (in_bom yes) (on_board yes) (fields_autoplaced)
@@
       (reference "R3") (unit 1) (value "680R") (footprint "Resistor_SMD:R_0402_1005Metric")
     )
+    (path "/f7fd3851-e44e-4431-8839-755499b365d7"
+      (reference "R4") (unit 1) (value "10K") (footprint "Resistor_SMD:R_0603_1608Metric")
+    )
     (path "/daf7af6f-f540-4fd4-a45d-1087a9c7bc20"
